File: host-usb.kicad_sch (KiCad schematic)
At the start: 20 parts, among them U1 CY7C68013A-56PVX, U2 24LC128, Y1 24MHz

Commit message: Add USB3343
Parts:
- added C14: 100nF, Capacitor_SMD:C_0402_1005Metric, symbol Device:C_Small
- added R7: 10K, Resistor_SMD:R_0402_1005Metric, symbol Device:R_Small
Connections:
- net +3V3: now also R7.1
- net GND: now also C14.2
- net ~{RESET}: now also C14.1, R7.2

Commit message: layout uncompleted
Parts:
- added TP10, TP11, TP12, TP9: Test, TestPoint:TestPoint_Pad_D1.0mm, symbol Connector:TestPoint
Connections:
- net +3V3: now also TP9.1
- net GND: now also TP12.1
- net ~{RESET}: now also TP11.1
- net A1: now reaches R2.2, U2.2 (A1)
- net A1: now also TP10.1
